Commit message: some corrections

File: model/bot.xacro (robot description, xacro)
@@ -8,5 +8,5 @@
   </xacro:macro>
 <!-- BASE_LINK PARAMETERS -->
-  <xacro:property name="bot_mass" value="30.0"/>
+  <xacro:property name="bot_mass" value="300.0"/>
   <xacro:property name="bot_width" value="0.75"/>
   <xacro:property name="bot_height" value="0.5"/>
@@ -15,4 +15,5 @@
   <xacro:property name="below_offset_btwn_base_wheel" value="0.02"/>
   <xacro:property name="wheel_thickness" value="0.02"/>
+  <xacro:property name="wheel_mass" value="0.2"/>
   <xacro:macro name="base_geometry">
     <geometry>
@@ -21,5 +22,5 @@
   </xacro:macro>
   <xacro:macro name="default_inertia">
-    <inertia ixx="0.6" ixy="0" ixz="0" iyy="0.65" iyz="0" izz="0.21"/>
+    <inertia ixx="4" ixy="0" ixz="0" iyy="4" iyz="0" izz="2"/>
   </xacro:macro>
 <!-- WHEEL PARAMETERS -->
@@ -52,38 +53,47 @@
         of the base_link-->
   <xacro:macro name="wheel" params="name *wheel_orientation *joint_orientation *joint_origin">
-    <joint name="${name}_base_joint" type="prismatic">
-      <parent link="base_link"/>
-      <child link="${name}_base_joint"/>
-      <limit effort="1000.0" lower="${-below_offset_btwn_base_wheel}" upper="${wheel_diameter}" velocity="0.2"/>
-      <xacro:insert_block name="joint_origin"/>
-      <axis xyz="0 0 1" rpy="0 0 0" />
-    </joint>
-    <joint name="${name}_wheel_joint" type="continuous">
-      <xacro:insert_block name="joint_orientation"/>
-      <parent link="${name}_base_joint"/>
-      <child link="${name}_wheel"/>
-      <!--xacro:insert_block name="origin_wheel"/-->
-      <!-- commented because origin of the wheels should be aligned with origin of the sliders -->
-      <origin xyz="0 0 0" rpy="0 0 0"/>
-    </joint>
-    <link name="${name}_wheel">
-      <visual>
-        <material name="black">
-          <color rgba="0 0 0 1"/>
-        </material>
-        <xacro:wheel_geometry_common/>
-        <xacro:insert_block name="wheel_orientation"/>
-      </visual>
-      <collision>
-        <xacro:wheel_geometry_common/>
-        <xacro:insert_block name="wheel_orientation"/>
-      </collision>
+    <link name="btwn_base_and_${name}wheel">
       <inertial>
-        <xacro:wheel_geometry_common/>
-        <xacro:insert_block name="wheel_orientation"/>
-        <mass value="${wheel_mass}"/>
-        <xacro:wheel_inertia/>
+        <mass value="${wheel_mass/3}" />
+        <origin xyz="0 0 0" />
+        <inertia ixx="0.1" ixy="0.0" ixz="0.0" iyy="0.1" iyz="0.0" izz="0.1"/>
       </inertial>
     </link>
+    <joint name="${name}_base_joint" type="prismatic">
+        <parent link="base_link"/>
+        <child link="btwn_base_and_${name}wheel"/>
+        <limit effort="100.0" lower="${-below_offset_btwn_base_wheel}" upper="${wheel_diameter}" velocity="100"/>
+        <xacro:insert_block name="joint_origin"/>
+        <axis xyz="0 0 1" rpy="0 0 0" />
+        <dynamics damping="0.7" friction="100000"/>
+        <safety_controller soft_lower_limit="-0.01"  soft_upper_limit="0.09" k_position="1" k_velocity="1"/>
+      </joint>
+    <link name="${name}_wheel">
+        <visual>
+          <material name="black">
+            <color rgba="0 0 0 1"/>
+          </material>
+          <xacro:wheel_geometry_common/>
+          <xacro:insert_block name="wheel_orientation"/>
+        </visual>
+        <collision>
+          <xacro:wheel_geometry_common/>
+          <xacro:insert_block name="wheel_orientation"/>
+        </collision>
+        <inertial>
+          <xacro:wheel_geometry_common/>
+          <xacro:insert_block name="wheel_orientation"/>
+          <mass value="${wheel_mass}"/>
+          <xacro:wheel_inertia/>
+        </inertial>
+    </link>
+    <joint name="${name}_wheel_joint" type="continuous">
+        <xacro:insert_block name="joint_orientation"/>
+        <parent link="btwn_base_and_${name}wheel"/>
+        <child link="${name}_wheel"/>
+        <!--xacro:insert_block name="origin_wheel"/-->
+        <!-- commented because origin of the wheels should be aligned with origin of the sliders -->
+        <origin xyz="0 0 0" rpy="0 0 0"/>
+    </joint>
       <!-- GAZEBO settings for wheels -->
     <gazebo reference="${name}_wheel">
@@ -91,8 +101,21 @@
       <mu2>1000000.0</mu2>
       <minDepth>0.0001 </minDepth>
-      <fdir1 value = "1 0 0"/>
+      <fdir1 value = "1 1 0"/>
       <kp>100000.0</kp>
       <kd>100000 </kd>
       <material>Gazebo/Black</material>
+      <selfCollide>0</selfCollide>
+      <gravity>0</gravity>
+    </gazebo>
+    <gazebo reference="btwn_base_and_${name}wheel">
+        <mu1>1000000.0</mu1>
+        <mu2>1000000.0</mu2>
+        <minDepth>0.0001 </minDepth>
+        <fdir1 value = "1 0 0"/>
+        <kp>100000.0</kp>
+        <kd>100000 </kd>
+        <material>Gazebo/Black</material>
+        <selfCollide>0</selfCollide>
+        <gravity>0</gravity>
     </gazebo>
   </xacro:macro>
@@ -104,4 +127,5 @@
       <mass value="${bot_mass}"/>
       <xacro:default_inertia/>
+      <xacro:base_geometry/>
     </inertial>
     <collision name='collision'>
@@ -115,46 +139,57 @@
   </link>
   <!-- WHEELS -->
-  <xacro:wheel name="1y">
-    <xacro:insert_block name="wheel_orientation_y"/>
-    <xacro:insert_block name="joint_axis_y"/>
+   <xacro:wheel name="1y">
+    <xacro:wheel_orientation_y/>
+    <xacro:joint_axis_y/>
     <origin xyz="${bot_width/2} ${-distance_between_wheels/2} ${-bot_height/2}" rpy="0 0 0"/>
   </xacro:wheel>
   <xacro:wheel name="2y">
-    <xacro:insert_block name="wheel_orientation_y"/>
-    <xacro:insert_block name="joint_axis_y"/>
+      <xacro:wheel_orientation_y/>
+      <xacro:joint_axis_y/>
     <origin xyz="${bot_width/2} ${distance_between_wheels/2} ${-bot_height/2}" rpy="0 0 0"/>
   </xacro:wheel>
   <xacro:wheel name="3y">
-    <xacro:insert_block name="wheel_orientation_y"/>
-    <xacro:insert_block name="joint_axis_y"/>
+      <xacro:wheel_orientation_y/>
+      <xacro:joint_axis_y/>
     <origin xyz="${-bot_width/2} ${-distance_between_wheels/2} ${-bot_height/2}" rpy="0 0 0"/>
   </xacro:wheel>
   <xacro:wheel name="4y">
-    <xacro:insert_block name="wheel_orientation_y"/>
-    <xacro:insert_block name="joint_axis_y"/>
+      <xacro:wheel_orientation_y/>
+      <xacro:joint_axis_y/>
     <origin xyz="${-bot_width/2} ${distance_between_wheels/2} ${-bot_height/2}" rpy="0 0 0"/>
   </xacro:wheel>
   <xacro:wheel name="5x">
-    <xacro:insert_block name="wheel_orientation_x"/>
-    <xacro:insert_block name="joint_axis_x"/>
+    <xacro:wheel_orientation_x/>
+    <xacro:joint_axis_x/>
     <origin xyz="${distance_between_wheels/2} ${bot_width/2 } ${-bot_height/2}" rpy="0 0 0"/>
   </xacro:wheel>
   <xacro:wheel name="6x">
-    <xacro:insert_block name="wheel_orientation_x"/>
-    <xacro:insert_block name="joint_axis_x"/>
+      <xacro:wheel_orientation_x/>
+      <xacro:joint_axis_x/>
     <origin xyz="${-distance_between_wheels/2} ${bot_width/2 } ${-bot_height/2}" rpy="0 0 0"/>
   </xacro:wheel>
   <xacro:wheel name="7x">
-    <xacro:insert_block name="wheel_orientation_x"/>
-    <xacro:insert_block name="joint_axis_x"/>
+      <xacro:wheel_orientation_x/>
+      <xacro:joint_axis_x/>
     <origin xyz="${distance_between_wheels/2} ${-bot_width/2 } ${-bot_height/2}" rpy="0 0 0"/>
   </xacro:wheel>
   <xacro:wheel name="8x">
-    <xacro:insert_block name="wheel_orientation_x"/>
-    <xacro:insert_block name="joint_axis_x"/>
+      <xacro:wheel_orientation_x/>
+      <xacro:joint_axis_x/>
     <origin xyz="${-distance_between_wheels/2} ${-bot_width/2 } ${-bot_height/2}" rpy="0 0 0"/>
   </xacro:wheel>
+  <gazebo reference="base_link">
+      <mu1>1000000.0</mu1>
+      <mu2>1000000.0</mu2>
+      <minDepth>0.0001 </minDepth>
+      <fdir1 value = "1 0 0"/>
+      <kp>100000.0</kp>
+      <kd>100000 </kd>
+      <material>Gazebo/Black</material>
+      <selfCollide>false</selfCollide>
+      <gravity>true</gravity>
+  </gazebo>
   <!-- LIDAR -->
-  <joint name="lidar_joint" type="fixed">
+  <!-- <joint name="lidar_joint" type="fixed">
     <axis xyz="0 0 0" />
     <origin xyz="${bot_length*6/7} 0 ${bot_height}" rpy="0 0 0"/>
@@ -180,7 +215,7 @@
       <inertia ixx="1e-6" ixy="0" ixz="0" iyy="1e-6" iyz="0" izz="1e-6" />
     </inertial>
-  </link>
+  </link>  -->
   <!-- GAZEBO PLUGINS -->
-  <gazebo>
+  <!-- <gazebo>
     <plugin name="differential_drive_controller" filename="libgazebo_ros_diff_drive.so">
       <alwaysOn>true</alwaysOn>
@@ -200,16 +235,6 @@
       <publishWheelJointState>true</publishWheelJointState>
     </plugin>
-  </gazebo>
-  <gazebo reference="ball">
-    <kp>1000000.0</kp>
-    <kd>10000</kd>
-    <dampingFactor>0.0</dampingFactor>
-    <mu1>0.00</mu1>
-    <mu2>0.00</mu2>
-    <fdir1 value = "1 0 0"/>
-    <maxVel>15.0</maxVel>
-    <material>Gazebo/Red</material>
-  </gazebo>
-  <gazebo reference="lidar">
+  </gazebo> -->
+  <!-- <gazebo reference="lidar">
     <sensor type="ray" name="head_hokuyo_sensor_front">
       <pose>0 0 0 0 0 0</pose>
@@ -223,5 +248,4 @@
             <min_angle>-1.3</min_angle>
             <max_angle>1.3</max_angle>
-            <!-- 1.570796 -->
           </horizontal>
         </scan>
@@ -233,8 +257,4 @@
         <noise>
           <type>gaussian</type>
-          <!-- Noise parameters based on published spec for Hokuyo laser
-               achieving "+-30mm" accuracy at range < 10m.  A mean of 0.0m and
-               stddev of 0.01m will put 99.7% of samples within 0.03m of the true
-               reading. -->
           <mean>0.0</mean>
           <stddev>0.01</stddev>
@@ -246,4 +266,4 @@
       </plugin>
     </sensor>
-  </gazebo>
+  </gazebo> -->
 </robot>

Commit message: Improvements

File: model/bot.xacro (robot description, xacro)
@@ -8,12 +8,12 @@
   </xacro:macro>
 <!-- BASE_LINK PARAMETERS -->
-  <xacro:property name="bot_mass" value="300.0"/>
+  <xacro:property name="bot_mass" value="30.0"/>
   <xacro:property name="bot_width" value="0.75"/>
   <xacro:property name="bot_height" value="0.5"/>
-  <xacro:property name="distance_between_wheels" value="0.6"/>
-  <xacro:property name="wheel_diameter" value="0.1" />
+  <xacro:property name="distance_between_wheels" value="0.5"/>
+  <xacro:property name="wheel_diameter" value="0.12" />
   <xacro:property name="below_offset_btwn_base_wheel" value="0.02"/>
-  <xacro:property name="wheel_thickness" value="0.02"/>
-  <xacro:property name="wheel_mass" value="0.2"/>
+  <xacro:property name="wheel_thickness" value="0.03"/>
+  <xacro:property name="wheel_mass" value="1"/>
   <xacro:macro name="base_geometry">
     <geometry>
@@ -26,5 +26,5 @@
 <!-- WHEEL PARAMETERS -->
   <xacro:macro name="wheel_inertia">
-      <inertia ixx="0.1" ixy="0.0" ixz="0.0" iyy="0.1" iyz="0.0" izz="0.1"/>
+      <inertia ixx="0.3" ixy="0.0" ixz="0.0" iyy="0.3" iyz="0.0" izz="0.3"/>
   </xacro:macro>
   <xacro:macro name="wheel_geometry_common">
@@ -55,18 +55,31 @@
     <link name="btwn_base_and_${name}wheel">
       <inertial>
-        <mass value="${wheel_mass/3}" />
+        <mass value="${wheel_mass/10}" />
         <origin xyz="0 0 0" />
-        <inertia ixx="0.1" ixy="0.0" ixz="0.0" iyy="0.1" iyz="0.0" izz="0.1"/>
+        <inertia ixx="0.01" ixy="0.0" ixz="0.0" iyy="0.01" iyz="0.0" izz="0.01"/>
       </inertial>
+      <visual>
+        <geometry>
+          <cylinder radius="0.01" length="0.01"/>
+        </geometry>
+        <origin xyz="0 0 0" rpy="0 0 0"/>
+      </visual>
+      <collision>
+        <geometry>
+          <cylinder radius="0.01" length="0.01"/>
+        </geometry>
+        <origin xyz="0 0 0" rpy="0 0 0"/>
+      </collision>
     </link>
     <joint name="${name}_base_joint" type="prismatic">
         <parent link="base_link"/>
         <child link="btwn_base_and_${name}wheel"/>
-        <limit effort="100.0" lower="${-below_offset_btwn_base_wheel}" upper="${wheel_diameter}" velocity="100"/>
+        <!-- <child link="${name}_wheel"/> -->
+        <limit effort="60.0" lower="${-below_offset_btwn_base_wheel-wheel_diameter}" upper="0.01" velocity="0.5"/>
         <xacro:insert_block name="joint_origin"/>
         <axis xyz="0 0 1" rpy="0 0 0" />
-        <dynamics damping="0.7" friction="100000"/>
-        <safety_controller soft_lower_limit="-0.01"  soft_upper_limit="0.09" k_position="1" k_velocity="1"/>
-      </joint>
+        <dynamics damping="0.3"/>
+        <safety_controller soft_lower_limit="-0.8" soft_upper_limit="0.1"  k_velocity="0.001" k_position="0.2"/>
+    </joint>
     <link name="${name}_wheel">
         <visual>
@@ -92,19 +105,17 @@
         <parent link="btwn_base_and_${name}wheel"/>
         <child link="${name}_wheel"/>
-        <!--xacro:insert_block name="origin_wheel"/-->
-        <!-- commented because origin of the wheels should be aligned with origin of the sliders -->
         <origin xyz="0 0 0" rpy="0 0 0"/>
     </joint>
       <!-- GAZEBO settings for wheels -->
     <gazebo reference="${name}_wheel">
-      <mu1>1000000.0</mu1>
-      <mu2>1000000.0</mu2>
-      <minDepth>0.0001 </minDepth>
-      <fdir1 value = "1 1 0"/>
-      <kp>100000.0</kp>
+      <mu1>10000000.0</mu1>
+      <mu2>10000000.0</mu2>
+      <minDepth>0.000001 </minDepth>
+      <fdir1 value = "1 0 0"/>
+      <kp>10000000.0</kp>
       <kd>100000 </kd>
       <material>Gazebo/Black</material>
       <selfCollide>0</selfCollide>
-      <gravity>0</gravity>
+      <gravity>1</gravity>
     </gazebo>
     <gazebo reference="btwn_base_and_${name}wheel">
@@ -119,4 +130,16 @@
         <gravity>0</gravity>
     </gazebo>
+    <!-- TRANSMISSION REQUIRED FOR PRISMATIC JOINTS TO WORK WITH PLUGINS -->
+    <transmission name="${name}_transmission">
+      <type>transmission_interface/SimpleTransmission</type>
+      <robotNamespace>/bot</robotNamespace>
+      <joint name="${name}_base_joint">
+        <hardwareInterface>hardware_interface/VelocityJointInterface</hardwareInterface>
+      </joint>
+      <actuator name="${name}_lift_motor">
+        <hardwareInterface>hardware_interface/VelocityJointInterface</hardwareInterface>
+        <mechanicalReduction>1</mechanicalReduction>
+      </actuator>
+    </transmission>
   </xacro:macro>
 <!-- DEFINITIONS OF ROBOT -->
@@ -142,40 +165,40 @@
     <xacro:wheel_orientation_y/>
     <xacro:joint_axis_y/>
-    <origin xyz="${bot_width/2} ${-distance_between_wheels/2} ${-bot_height/2}" rpy="0 0 0"/>
+    <origin xyz="${bot_width/2} ${-distance_between_wheels/2} ${-bot_height/2+wheel_diameter/3*2}" rpy="0 0 0"/>
   </xacro:wheel>
   <xacro:wheel name="2y">
       <xacro:wheel_orientation_y/>
       <xacro:joint_axis_y/>
-    <origin xyz="${bot_width/2} ${distance_between_wheels/2} ${-bot_height/2}" rpy="0 0 0"/>
+    <origin xyz="${bot_width/2} ${distance_between_wheels/2} ${-bot_height/2+wheel_diameter/3*2}" rpy="0 0 0"/>
   </xacro:wheel>
   <xacro:wheel name="3y">
       <xacro:wheel_orientation_y/>
       <xacro:joint_axis_y/>
-    <origin xyz="${-bot_width/2} ${-distance_between_wheels/2} ${-bot_height/2}" rpy="0 0 0"/>
+    <origin xyz="${-bot_width/2} ${-distance_between_wheels/2} ${-bot_height/2+wheel_diameter/3*2}" rpy="0 0 0"/>
   </xacro:wheel>
   <xacro:wheel name="4y">
       <xacro:wheel_orientation_y/>
       <xacro:joint_axis_y/>
-    <origin xyz="${-bot_width/2} ${distance_between_wheels/2} ${-bot_height/2}" rpy="0 0 0"/>
+    <origin xyz="${-bot_width/2} ${distance_between_wheels/2} ${-bot_height/2+wheel_diameter/3*2}" rpy="0 0 0"/>
   </xacro:wheel>
   <xacro:wheel name="5x">
     <xacro:wheel_orientation_x/>
     <xacro:joint_axis_x/>
-    <origin xyz="${distance_between_wheels/2} ${bot_width/2 } ${-bot_height/2}" rpy="0 0 0"/>
+    <origin xyz="${distance_between_wheels/2} ${bot_width/2 } ${-bot_height/2+wheel_diameter/3*2}" rpy="0 0 0"/>
   </xacro:wheel>
   <xacro:wheel name="6x">
       <xacro:wheel_orientation_x/>
       <xacro:joint_axis_x/>
-    <origin xyz="${-distance_between_wheels/2} ${bot_width/2 } ${-bot_height/2}" rpy="0 0 0"/>
+    <origin xyz="${-distance_between_wheels/2} ${bot_width/2 } ${-bot_height/2+wheel_diameter/3*2}" rpy="0 0 0"/>
   </xacro:wheel>
   <xacro:wheel name="7x">
       <xacro:wheel_orientation_x/>
       <xacro:joint_axis_x/>
-    <origin xyz="${distance_between_wheels/2} ${-bot_width/2 } ${-bot_height/2}" rpy="0 0 0"/>
+    <origin xyz="${distance_between_wheels/2} ${-bot_width/2 } ${-bot_height/2+wheel_diameter/3*2}" rpy="0 0 0"/>
   </xacro:wheel>
   <xacro:wheel name="8x">
       <xacro:wheel_orientation_x/>
       <xacro:joint_axis_x/>
-    <origin xyz="${-distance_between_wheels/2} ${-bot_width/2 } ${-bot_height/2}" rpy="0 0 0"/>
+    <origin xyz="${-distance_between_wheels/2} ${-bot_width/2 } ${-bot_height/2+wheel_diameter/3*2}" rpy="0 0 0"/>
   </xacro:wheel>
   <gazebo reference="base_link">
@@ -184,6 +207,6 @@
       <minDepth>0.0001 </minDepth>
       <fdir1 value = "1 0 0"/>
-      <kp>100000.0</kp>
-      <kd>100000 </kd>
+      <kp>10000.0</kp>
+      <kd>10000 </kd>
       <material>Gazebo/Black</material>
       <selfCollide>false</selfCollide>
@@ -216,16 +239,32 @@
     </inertial>
   </link>  -->
+  <gazebo>
+    <plugin name="gazebo_ros_control" filename="libgazebo_ros_control.so">
+      <robotNamespace>/bot</robotNamespace>
+      <robotSimType>gazebo_ros_control/DefaultRobotHWSim</robotSimType>
+    </plugin>
+  </gazebo>
   <!-- GAZEBO PLUGINS -->
-  <!-- <gazebo>
+  <gazebo>
     <plugin name="differential_drive_controller" filename="libgazebo_ros_diff_drive.so">
       <alwaysOn>true</alwaysOn>
       <publishTf>1</publishTf>
       <updateRate>50</updateRate>
-      <leftJoint>left_wheel_joint</leftJoint>
-      <rightJoint>right_wheel_joint</rightJoint>
-      <wheelSeparation>0.2</wheelSeparation>
-      <wheelDiameter>0.05</wheelDiameter>
-      <torque>75</torque>
-      <commandTopic>cmd_vel</commandTopic>
+      <leftJoint>1y_wheel_joint</leftJoint>
+      <rightJoint>3y_wheel_joint</rightJoint>
+      <wheelSeparation>0.75</wheelSeparation>
+      <angular>
+        <z>
+          <has_velocity_limits>true</has_velocity_limits>
+          <max_velocity>0</max_velocity>
+          <has_acceleration_limits>true</has_acceleration_limits>
+          <max_acceleration>0</max_acceleration>
+          <has_jerk_limits>true</has_jerk_limits>
+          <max_jerk>0</max_jerk>
+        </z>
+      </angular>
+      <wheelDiameter>0.12</wheelDiameter>
+      <torque>120</torque>
+      <commandTopic>cmd_vel_x</commandTopic>
       <odometryTopic>odom</odometryTopic>
       <odometryFrame>odom</odometryFrame>
@@ -235,5 +274,5 @@
       <publishWheelJointState>true</publishWheelJointState>
     </plugin>
-  </gazebo> -->
+  </gazebo>
   <!-- <gazebo reference="lidar">
     <sensor type="ray" name="head_hokuyo_sensor_front">
