Commit message: stability

File: model/bot.xacro (robot description, xacro)
@@ -45,4 +45,32 @@
     <axis xyz="1 0 0" rpy="0 0 0" />
   </xacro:macro>
+  <!-- friction is high so these wheels are drivers -->
+  <xacro:macro name="primary_wheel_physical_params" params="wheel_name">
+    <gazebo reference="${wheel_name}_wheel">
+        <mu1>10000.0</mu1>
+        <mu2>10000.0</mu2>
+        <minDepth>0.0001 </minDepth>
+        <fdir1 value = "0 0 0"/>
+        <kp>2147483647.0</kp>
+        <kd>1.0 </kd>
+        <material>Gazebo/Black</material>
+        <selfCollide>0</selfCollide>
+        <gravity>1</gravity>
+        <max_vel>0.0001</max_vel>
+      </gazebo>
+  </xacro:macro>
+  <!-- friction is low so these wheels are casters -->
+  <xacro:macro name="secondary_wheel_physical_params" params="wheel_name">
+    <gazebo reference="${wheel_name}_wheel">
+        <material>Gazebo/Black</material>
+        <kp>2147483647.0</kp>
+        <kd>1.0</kd>
+        <dampingFactor>0.0</dampingFactor>
+        <mu1>0.00</mu1>
+        <mu2>0.00</mu2>
+        <fdir1 value = "0 0 0"/>
+        <maxVel>15.0</maxVel>
+      </gazebo>
+  </xacro:macro>
   <!-- origin_wheel - location of where the wheel is attached
         wheel_orientation - the direction (axis) of where the wheel is turned straight to
@@ -51,6 +79,7 @@
         so wheel_orientation is x, joint_orientation is x
         joint_origin - the location of where the slider joint is attached (should be at the very edge of the bottom
-        of the base_link-->
-  <xacro:macro name="wheel" params="name *wheel_orientation *joint_orientation *joint_origin">
+        of the base_link
+      -->
+  <xacro:macro name="wheel" params="name *wheel_orientation *joint_orientation *joint_origin *wheel_physical_params">
     <link name="btwn_base_and_${name}wheel">
       <inertial>
@@ -76,10 +105,14 @@
         <child link="btwn_base_and_${name}wheel"/>
         <!-- <child link="${name}_wheel"/> -->
-        <limit effort="60.0" lower="${-below_offset_btwn_base_wheel-wheel_diameter}" upper="0.01" velocity="0.5"/>
+        <limit effort="200.0" lower="${-below_offset_btwn_base_wheel-wheel_diameter}" upper="0.01" velocity="0.5"/>
         <xacro:insert_block name="joint_origin"/>
         <axis xyz="0 0 1" rpy="0 0 0" />
-        <dynamics damping="0.3"/>
+        <!-- little damping reduces some oscillations a bit -->
+        <dynamics damping="0.05"/>
+        <!-- lower and upper limits should be slightly less than those mentioned in <joint> tag
+            k_velocity should be small - less oscillations, k_position can be a bit higher but it influences
+            more on speed of joint moving than on oscillations -->
         <safety_controller soft_lower_limit="-0.8" soft_upper_limit="0.1"  k_velocity="0.001" k_position="0.2"/>
-    </joint>
+      </joint>
     <link name="${name}_wheel">
         <visual>
@@ -108,15 +141,6 @@
     </joint>
       <!-- GAZEBO settings for wheels -->
-    <gazebo reference="${name}_wheel">
-      <mu1>10000000.0</mu1>
-      <mu2>10000000.0</mu2>
-      <minDepth>0.000001 </minDepth>
-      <fdir1 value = "1 0 0"/>
-      <kp>10000000.0</kp>
-      <kd>100000 </kd>
-      <material>Gazebo/Black</material>
-      <selfCollide>0</selfCollide>
-      <gravity>1</gravity>
-    </gazebo>
+      <!-- on each side of the robot should be 2 driver wheels and 2 non-driver caster wheels so they don't conflict -->
+    <xacro:insert_block name="wheel_physical_params"/>
     <gazebo reference="btwn_base_and_${name}wheel">
         <mu1>1000000.0</mu1>
@@ -166,19 +190,23 @@
     <xacro:joint_axis_y/>
     <origin xyz="${bot_width/2} ${-distance_between_wheels/2} ${-bot_height/2+wheel_diameter/3*2}" rpy="0 0 0"/>
+    <xacro:primary_wheel_physical_params wheel_name="1y"/>
   </xacro:wheel>
   <xacro:wheel name="2y">
-      <xacro:wheel_orientation_y/>
-      <xacro:joint_axis_y/>
+    <xacro:wheel_orientation_y/>
+    <xacro:joint_axis_y/>
     <origin xyz="${bot_width/2} ${distance_between_wheels/2} ${-bot_height/2+wheel_diameter/3*2}" rpy="0 0 0"/>
+    <xacro:secondary_wheel_physical_params wheel_name="2y"/>
   </xacro:wheel>
   <xacro:wheel name="3y">
-      <xacro:wheel_orientation_y/>
-      <xacro:joint_axis_y/>
+    <xacro:wheel_orientation_y/>
+    <xacro:joint_axis_y/>
     <origin xyz="${-bot_width/2} ${-distance_between_wheels/2} ${-bot_height/2+wheel_diameter/3*2}" rpy="0 0 0"/>
+    <xacro:primary_wheel_physical_params wheel_name="3y"/>
   </xacro:wheel>
   <xacro:wheel name="4y">
-      <xacro:wheel_orientation_y/>
-      <xacro:joint_axis_y/>
+    <xacro:wheel_orientation_y/>
+    <xacro:joint_axis_y/>
     <origin xyz="${-bot_width/2} ${distance_between_wheels/2} ${-bot_height/2+wheel_diameter/3*2}" rpy="0 0 0"/>
+    <xacro:secondary_wheel_physical_params wheel_name="4y"/>
   </xacro:wheel>
   <xacro:wheel name="5x">
@@ -186,19 +214,23 @@
     <xacro:joint_axis_x/>
     <origin xyz="${distance_between_wheels/2} ${bot_width/2 } ${-bot_height/2+wheel_diameter/3*2}" rpy="0 0 0"/>
+    <xacro:primary_wheel_physical_params wheel_name="5x"/>
   </xacro:wheel>
   <xacro:wheel name="6x">
-      <xacro:wheel_orientation_x/>
-      <xacro:joint_axis_x/>
+    <xacro:wheel_orientation_x/>
+    <xacro:joint_axis_x/>
     <origin xyz="${-distance_between_wheels/2} ${bot_width/2 } ${-bot_height/2+wheel_diameter/3*2}" rpy="0 0 0"/>
+    <xacro:secondary_wheel_physical_params wheel_name="6x"/>
   </xacro:wheel>
   <xacro:wheel name="7x">
-      <xacro:wheel_orientation_x/>
-      <xacro:joint_axis_x/>
+    <xacro:wheel_orientation_x/>
+    <xacro:joint_axis_x/>
     <origin xyz="${distance_between_wheels/2} ${-bot_width/2 } ${-bot_height/2+wheel_diameter/3*2}" rpy="0 0 0"/>
+    <xacro:primary_wheel_physical_params wheel_name="7x"/>
   </xacro:wheel>
   <xacro:wheel name="8x">
-      <xacro:wheel_orientation_x/>
-      <xacro:joint_axis_x/>
+    <xacro:wheel_orientation_x/>
+    <xacro:joint_axis_x/>
     <origin xyz="${-distance_between_wheels/2} ${-bot_width/2 } ${-bot_height/2+wheel_diameter/3*2}" rpy="0 0 0"/>
+    <xacro:secondary_wheel_physical_params wheel_name="8x"/>
   </xacro:wheel>
   <gazebo reference="base_link">
@@ -213,30 +245,5 @@
       <gravity>true</gravity>
   </gazebo>
-  <!-- LIDAR -->
-  <!-- <joint name="lidar_joint" type="fixed">
-    <axis xyz="0 0 0" />
-    <origin xyz="${bot_length*6/7} 0 ${bot_height}" rpy="0 0 0"/>
-    <parent link="base_link"/>
-    <child link="lidar"/>
-  </joint>
-  <link name="lidar">
-    <collision>
-      <origin xyz="0 0 0" rpy="0 0 0"/>
-      <geometry>
-        <box size="0.03 0.03 0.03"/>
-      </geometry>
-    </collision>
-    <visual>
-      <origin xyz="0 0 0" rpy="0 0 0"/>
-      <geometry>
-        <box size="0.03 0.03 0.03"/>
-      </geometry>
-    </visual>
-    <inertial>
-      <mass value="1e-5" />
-      <origin xyz="0 0 0" rpy="0 0 0"/>
-      <inertia ixx="1e-6" ixy="0" ixz="0" iyy="1e-6" iyz="0" izz="1e-6" />
-    </inertial>
-  </link>  -->
+  <!-- should be turned on because we are using some interfaces to control joints -->
   <gazebo>
     <plugin name="gazebo_ros_control" filename="libgazebo_ros_control.so">
@@ -246,4 +253,5 @@
   </gazebo>
   <!-- GAZEBO PLUGINS -->
+  <!-- setup of 4 driver primary wheels -->
   <gazebo>
     <plugin name="differential_drive_controller" filename="libgazebo_ros_diff_drive.so">
@@ -253,4 +261,33 @@
       <leftJoint>1y_wheel_joint</leftJoint>
       <rightJoint>3y_wheel_joint</rightJoint>
+      <wheelSeparation>0.75</wheelSeparation>
+      <angular>
+        <z>
+          <has_velocity_limits>true</has_velocity_limits>
+          <max_velocity>0</max_velocity>
+          <has_acceleration_limits>true</has_acceleration_limits>
+          <max_acceleration>0</max_acceleration>
+          <has_jerk_limits>true</has_jerk_limits>
+          <max_jerk>0</max_jerk>
+        </z>
+      </angular>
+      <wheelDiameter>0.12</wheelDiameter>
+      <torque>120</torque>
+      <commandTopic>cmd_vel_y</commandTopic>
+      <odometryTopic>odom</odometryTopic>
+      <odometryFrame>odom</odometryFrame>
+      <robotBaseFrame>base_link</robotBaseFrame>
+      <odometrySource>world</odometrySource>
+      <publishWheelTF>true</publishWheelTF>
+      <publishWheelJointState>true</publishWheelJointState>
+    </plugin>
+  </gazebo>
+  <gazebo>
+    <plugin name="differential_drive_controller_2" filename="libgazebo_ros_diff_drive.so">
+      <alwaysOn>true</alwaysOn>
+      <publishTf>1</publishTf>
+      <updateRate>50</updateRate>
+      <leftJoint>5x_wheel_joint</leftJoint>
+      <rightJoint>7x_wheel_joint</rightJoint>
       <wheelSeparation>0.75</wheelSeparation>
       <angular>
@@ -275,34 +312,3 @@
     </plugin>
   </gazebo>
-  <!-- <gazebo reference="lidar">
-    <sensor type="ray" name="head_hokuyo_sensor_front">
-      <pose>0 0 0 0 0 0</pose>
-      <visualize>true</visualize>
-      <update_rate>40</update_rate>
-      <ray>
-        <scan>
-          <horizontal>
-            <samples>720</samples>
-            <resolution>1</resolution>
-            <min_angle>-1.3</min_angle>
-            <max_angle>1.3</max_angle>
-          </horizontal>
-        </scan>
-        <range>
-          <min>0.1</min>
-          <max>30.0</max>
-          <resolution>0.01</resolution>
-        </range>
-        <noise>
-          <type>gaussian</type>
-          <mean>0.0</mean>
-          <stddev>0.01</stddev>
-        </noise>
-      </ray>
-      <plugin name="gazebo_ros_head_hokuyo_controller" filename="libgazebo_ros_laser.so">
-        <topicName>scan</topicName>
-        <frameName>lidar</frameName>
-      </plugin>
-    </sensor>
-  </gazebo> -->
 </robot>

Commit message: working version of server

File: model/bot.xacro (robot description, xacro)
@@ -15,5 +15,5 @@
   <xacro:property name="below_offset_btwn_base_wheel" value="0.02"/>
   <xacro:property name="wheel_thickness" value="0.03"/>
-  <xacro:property name="wheel_mass" value="1"/>
+  <xacro:property name="wheel_mass" value="0.3"/>
   <xacro:macro name="base_geometry">
     <geometry>
@@ -21,14 +21,31 @@
     </geometry>
   </xacro:macro>
+  <macro name="cylinder_inertia" params="m r h">
+    <inertia  ixx="${m*(3*r*r+h*h)/12}" ixy = "0" ixz = "0"
+      iyy="${m*(3*r*r+h*h)/12}" iyz = "0"
+      izz="${m*r*r/2}"
+    />
+  </macro>
+ <macro name="box_inertia" params="m x y z">
+    <inertia  ixx="${m*(y*y+z*z)/12}" ixy = "0" ixz = "0"
+      iyy="${m*(x*x+z*z)/12}" iyz = "0"
+      izz="${m*(x*x+z*z)/12}"
+    />
+  </macro>
   <xacro:macro name="default_inertia">
-    <inertia ixx="4" ixy="0" ixz="0" iyy="4" iyz="0" izz="2"/>
+    <box_inertia m="${bot_mass}" x="${bot_width}" y="${bot_width}" z="${bot_height}"/>
   </xacro:macro>
 <!-- WHEEL PARAMETERS -->
   <xacro:macro name="wheel_inertia">
-      <inertia ixx="0.3" ixy="0.0" ixz="0.0" iyy="0.3" iyz="0.0" izz="0.3"/>
+    <cylinder_inertia m="${wheel_mass}" r="${wheel_diameter/2}" h="${0.01}"/>
   </xacro:macro>
   <xacro:macro name="wheel_geometry_common">
       <geometry>
-          <cylinder radius="${wheel_diameter/2}" length="${wheel_thickness}"/>
+          <cylinder radius="${wheel_diameter/2}" length="${wheel_thickness/3}"/>
+      </geometry>
+  </xacro:macro>
+  <xacro:macro name="wheel_smooth_geometry">
+      <geometry>
+          <mesh filename="file://$(arg meshDirectory)/mesh/wheel_smooth.stl" scale="0.01 0.01 0.01"/>
       </geometry>
   </xacro:macro>
@@ -37,5 +54,11 @@
   </xacro:macro>
   <xacro:macro name="wheel_orientation_y">
-    <origin xyz="0 0 0" rpy="0 ${pi/2} 0"/>
+    <origin xyz="0 0 0" rpy="0 ${pi/2} ${pi}"/>
+  </xacro:macro>
+  <xacro:macro name="wheel_smooth_orientation_x">
+    <origin xyz="0 0 0" rpy="${pi/2} ${pi/2} ${pi/2}"/>
+  </xacro:macro>
+  <xacro:macro name="wheel_smooth_orientation_y">
+    <origin xyz="0 0 0" rpy="${pi/2} ${pi/2} 0"/>
   </xacro:macro>
   <xacro:macro name="joint_axis_x">
@@ -43,16 +66,16 @@
   </xacro:macro>
   <xacro:macro name="joint_axis_y">
-    <axis xyz="1 0 0" rpy="0 0 0" />
+    <axis xyz="-1 0 0" rpy="0 0 0" />
   </xacro:macro>
   <!-- friction is high so these wheels are drivers -->
   <xacro:macro name="primary_wheel_physical_params" params="wheel_name">
     <gazebo reference="${wheel_name}_wheel">
-        <mu1>1000000.0</mu1>
-        <mu2>1000000.0</mu2>
-        <fdir1 value = "1 1 0"/>
-        <kp>2147483647.0</kp>
-        <kd>1.0 </kd>
+        <mu1>100000.0</mu1>
+        <mu2>100000.0</mu2>
+        <fdir1 value = "0 0 0"/>
+        <kp>1e+13</kp>
+        <kd>1000</kd>
         <material>Gazebo/Black</material>
-        <minDepth>0.01 </minDepth>
+        <minDepth>0.0001 </minDepth>
       </gazebo>
   </xacro:macro>
@@ -61,10 +84,10 @@
     <gazebo reference="${wheel_name}_wheel">
         <material>Gazebo/Black</material>
-        <kp>2147483647.0</kp>
-        <kd>1.0</kd>
-        <mu1>100.00</mu1>
-        <mu2>100.00</mu2>
-        <fdir1 value = "1 1 0"/>
-        <minDepth>0.01 </minDepth>
+        <kp>1e+13</kp>
+        <kd>1000</kd>
+        <mu1>0.00</mu1>
+        <mu2>0.00</mu2>
+        <fdir1 value = "0 0 0"/>
+        <minDepth>0.0001 </minDepth>
       </gazebo>
   </xacro:macro>
@@ -77,5 +100,5 @@
         of the base_link
       -->
-  <xacro:macro name="wheel" params="name *wheel_orientation *joint_orientation *joint_origin *wheel_physical_params">
+  <xacro:macro name="wheel" params="name *wheel_orientation *joint_orientation *joint_origin *wheel_physical_params *wheel_smooth_orientation">
     <link name="btwn_base_and_${name}wheel">
       <inertial>
@@ -126,5 +149,5 @@
           <xacro:wheel_geometry_common/>
           <xacro:insert_block name="wheel_orientation"/>
-          <mass value="${wheel_mass}"/>
+          <mass value="${wheel_mass/2}"/>
           <xacro:wheel_inertia/>
         </inertial>
@@ -136,18 +159,54 @@
         <origin xyz="0 0 0" rpy="0 0 0"/>
     </joint>
+    <link name="${name}_wheel_smooth">
+      <visual>
+        <material name="cyan">
+          <color rgba="0 255 255 1"/>
+        </material>
+        <xacro:wheel_smooth_geometry/>
+        <xacro:insert_block name="wheel_smooth_orientation"/>
+      </visual>
+      <collision>
+        <xacro:wheel_smooth_geometry/>
+        <xacro:insert_block name="wheel_smooth_orientation"/>
+      </collision>
+      <inertial>
+        <xacro:wheel_smooth_geometry/>
+        <xacro:insert_block name="wheel_smooth_orientation"/>
+        <mass value="${wheel_mass}"/>
+        <xacro:wheel_inertia/>
+      </inertial>
+  </link>
+  <joint name="${name}_wheel__wheel_smooth" type="revolute" >
+    <limit upper="0.0" lower="0.0" effort="1000.0" velocity="0.0"/>
+    <parent link="${name}_wheel"/>
+    <child link="${name}_wheel_smooth"/>
+    <origin xyz="0 0 0" rpy="0 0 0"/>
+  </joint>
       <!-- GAZEBO settings for wheels -->
       <!-- on each side of the robot should be 2 driver wheels and 2 non-driver caster wheels so they don't conflict -->
     <xacro:insert_block name="wheel_physical_params"/>
     <gazebo reference="btwn_base_and_${name}wheel">
-        <mu1>1000000.0</mu1>
-        <mu2>1000000.0</mu2>
+        <mu1>100.0</mu1>
+        <mu2>100.0</mu2>
         <minDepth>0.0001 </minDepth>
         <fdir1 value = "1 0 0"/>
         <kp>100000.0</kp>
-        <kd>100000 </kd>
+        <kd>1000 </kd>
         <material>Gazebo/Black</material>
         <selfCollide>0</selfCollide>
         <gravity>0</gravity>
     </gazebo>
+    <gazebo reference="${name}_wheel_smooth">
+        <material>Gazebo/Blue</material>
+        <mu1>0.0</mu1>
+        <mu2>0.0</mu2>
+        <minDepth>0.0000 </minDepth>
+        <fdir1 value = "0 0 0"/>
+        <kp>100000.0</kp>
+        <kd>1000 </kd>
+        <selfCollide>0</selfCollide>
+        <gravity>1</gravity>
+      </gazebo>
     <!-- TRANSMISSION REQUIRED FOR PRISMATIC JOINTS TO WORK WITH PLUGINS -->
     <transmission name="${name}_transmission">
@@ -187,4 +246,5 @@
     <origin xyz="${bot_width/2} ${-distance_between_wheels/2} ${-bot_height/2+wheel_diameter/3*2}" rpy="0 0 0"/>
     <xacro:primary_wheel_physical_params wheel_name="1y"/>
+    <xacro:wheel_smooth_orientation_y/>
   </xacro:wheel>
   <xacro:wheel name="2y">
@@ -193,4 +253,5 @@
     <origin xyz="${bot_width/2} ${distance_between_wheels/2} ${-bot_height/2+wheel_diameter/3*2}" rpy="0 0 0"/>
     <xacro:secondary_wheel_physical_params wheel_name="2y"/>
+    <xacro:wheel_smooth_orientation_y/>
   </xacro:wheel>
   <xacro:wheel name="3y">
@@ -199,4 +260,5 @@
     <origin xyz="${-bot_width/2} ${-distance_between_wheels/2} ${-bot_height/2+wheel_diameter/3*2}" rpy="0 0 0"/>
     <xacro:primary_wheel_physical_params wheel_name="3y"/>
+    <xacro:wheel_smooth_orientation_y/>
   </xacro:wheel>
   <xacro:wheel name="4y">
@@ -205,4 +267,5 @@
     <origin xyz="${-bot_width/2} ${distance_between_wheels/2} ${-bot_height/2+wheel_diameter/3*2}" rpy="0 0 0"/>
     <xacro:secondary_wheel_physical_params wheel_name="4y"/>
+    <xacro:wheel_smooth_orientation_y/>
   </xacro:wheel>
   <xacro:wheel name="5x">
@@ -211,4 +274,5 @@
     <origin xyz="${distance_between_wheels/2} ${bot_width/2 } ${-bot_height/2+wheel_diameter/3*2}" rpy="0 0 0"/>
     <xacro:primary_wheel_physical_params wheel_name="5x"/>
+    <xacro:wheel_smooth_orientation_x/>
   </xacro:wheel>
   <xacro:wheel name="6x">
@@ -217,4 +281,5 @@
     <origin xyz="${-distance_between_wheels/2} ${bot_width/2 } ${-bot_height/2+wheel_diameter/3*2}" rpy="0 0 0"/>
     <xacro:secondary_wheel_physical_params wheel_name="6x"/>
+    <xacro:wheel_smooth_orientation_x/>
   </xacro:wheel>
   <xacro:wheel name="7x">
@@ -223,4 +288,5 @@
     <origin xyz="${distance_between_wheels/2} ${-bot_width/2 } ${-bot_height/2+wheel_diameter/3*2}" rpy="0 0 0"/>
     <xacro:primary_wheel_physical_params wheel_name="7x"/>
+    <xacro:wheel_smooth_orientation_x/>
   </xacro:wheel>
   <xacro:wheel name="8x">
@@ -229,4 +295,5 @@
     <origin xyz="${-distance_between_wheels/2} ${-bot_width/2 } ${-bot_height/2+wheel_diameter/3*2}" rpy="0 0 0"/>
     <xacro:secondary_wheel_physical_params wheel_name="8x"/>
+    <xacro:wheel_smooth_orientation_x/>
   </xacro:wheel>
   <gazebo reference="base_link">
@@ -254,7 +321,7 @@
       <alwaysOn>true</alwaysOn>
       <publishTf>1</publishTf>
-      <updateRate>50</updateRate>
-      <leftJoint>1y_wheel_joint</leftJoint>
-      <rightJoint>3y_wheel_joint</rightJoint>
+      <updateRate>100</updateRate>
+      <leftJoint>3y_wheel_joint</leftJoint>
+      <rightJoint>1y_wheel_joint</rightJoint>
       <wheelSeparation>0.75</wheelSeparation>
       <angular>
@@ -269,5 +336,5 @@
       </angular>
       <wheelDiameter>0.12</wheelDiameter>
-      <torque>120</torque>
+      <torque>300</torque>
       <commandTopic>cmd_vel_y</commandTopic>
       <odometryTopic>odom</odometryTopic>
@@ -283,5 +350,5 @@
       <alwaysOn>true</alwaysOn>
       <publishTf>1</publishTf>
-      <updateRate>50</updateRate>
+      <updateRate>100</updateRate>
       <leftJoint>5x_wheel_joint</leftJoint>
       <rightJoint>7x_wheel_joint</rightJoint>
@@ -298,5 +365,5 @@
       </angular>
       <wheelDiameter>0.12</wheelDiameter>
-      <torque>120</torque>
+      <torque>500</torque>
       <commandTopic>cmd_vel_x</commandTopic>
       <odometryTopic>odom</odometryTopic>

Commit message: Velocity limits increased

File: model/bot.xacro (robot description, xacro)
@@ -124,5 +124,5 @@
         <child link="btwn_base_and_${name}wheel"/>
         <!-- <child link="${name}_wheel"/> -->
-        <limit effort="200.0" lower="${-below_offset_btwn_base_wheel-wheel_diameter}" upper="0.01" velocity="0.5"/>
+        <limit effort="200.0" lower="${-below_offset_btwn_base_wheel-wheel_diameter}" upper="0.01" velocity="2"/>
         <xacro:insert_block name="joint_origin"/>
         <axis xyz="0 0 1" rpy="0 0 0" />
@@ -132,5 +132,5 @@
             k_velocity should be small - less oscillations, k_position can be a bit higher but it influences
             more on speed of joint moving than on oscillations -->
-        <safety_controller soft_lower_limit="-0.8" soft_upper_limit="0.1"  k_velocity="0.001" k_position="0.2"/>
+        <safety_controller soft_lower_limit="-0.8" soft_upper_limit="0.1"  k_velocity="0.01" k_position="0.2"/>
       </joint>
     <link name="${name}_wheel">
